File: Home Control/Hardware/PCB Design/Board/Home_Control.sch (EAGLE design)
At the start: 30 parts, among them J1 282837-3, J3 282837-3, P1 282837-2, P2 282837-2, P3 282837-2, P4 282837-2, P5 282837-2, T1 BT138-V, T2 BT138-V, T3 BT138-V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

Commit message: Add files via upload
Other:
- note added: "Home control board for contolling 4 AC devices by triac using PIR, LDR and DHT11"
- note removed: "Home control board for contolling 4 AC devices by triac using PIR and 2 LDR"
Changed lines of the file:
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@@
 <text x="88.9" y="10.16" size="2.1844" layer="94">Home control board
 for contolling 4 AC devices by triac
-using PIR and 2 LDR</text>
+using PIR, LDR and DHT11</text>
 <wire x1="142.24" y1="86.36" x2="180.34" y2="86.36" width="0.1524" layer="94"/>
 <wire x1="43.18" y1="3.81" x2="43.18" y2="24.13" width="0.1524" layer="94"/>
